File: hard/DebuggerKB.brd (EAGLE design)
At the start: 110 x 70 mm, 26 parts, among them CN1 PH-2, Q1 DTC014EEB, Q2 TPC8125, SW1 CL-SA-12C4, SW10 CHERRY-MX, SW11 CHERRY-MX, SW12 CHERRY-MX, SW2 CHERRY-MX, SW3 CHERRY-MX, SW4 CHERRY-MX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

Commit message: modify board design
Parts:
- CN2: value (none) -> PINHD
- SW10, SW11, SW12, SW2, SW3, SW4, SW5, SW6, SW7, SW8, SW9: value CHERRY-MX -> KAILH_SWITCH_SOCKET; device lipoyang_mechanical:CHERRY-MX -> lipoyang_mechanical:SWITCH_SOCKET
- moved D3 10.3 mm to (105.0, 37.5)
- moved D4 8.00 mm to (103.0, 20.0)
Routing:
- net N$6: track 96.0 -> 117.2 mm
- net N$5: track 96.0 -> 116.0 mm
- net OUT2: track 66.9 -> 47.4 mm
- net IN4: track 71.1 -> 79.7 mm, vias 1 -> 3
- net IN3: track 91.9 -> 99.9 mm, vias 1 -> 3
- net IN2: track 112.6 -> 120.3 mm, vias 1 -> 3
- net IN1: track 133.4 -> 140.8 mm, vias 1 -> 3
- net IN5: track 59.0 -> 54.0 mm, vias 1 -> 3
- net PAGE_SW: track 63.2 -> 59.4 mm
- net OUT1: track 35.1 -> 33.3 mm
