File: hard/DebuggerKB.sch (EAGLE design)
At the start: 26 parts, among them CN1 PH-2, Q1 DTC014EEB, Q2 TPC8125, SW1 CL-SA-12C4, SW10 CHERRY-MX, SW11 CHERRY-MX, SW12 CHERRY-MX, SW2 CHERRY-MX, SW3 CHERRY-MX, SW4 CHERRY-MX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

Commit message: modify board design
Parts:
- CN2: value (none) -> PINHD
- SW10, SW11, SW12, SW2, SW3, SW4, SW5, SW6, SW7, SW8, SW9: value CHERRY-MX -> KAILH_SWITCH_SOCKET; device lipoyang_mechanical:CHERRY-MX -> lipoyang_mechanical:KAILH_SWITCH_SOCKET
Other:
- moved on the sheet: SW10, SW11, SW12, SW2, SW3, SW4, SW5, SW6, SW7, SW8, SW9
